File: Marv-Atreus.kicad_pcb (KiCad board)
At the start: 2 copper layers, 240.3 x 101.9 mm, 102 parts, among them SW1 SW_Push, U1 ATmega32U4-AU, Y1 16MHz

Commit message: Rerotued the board
Parts:
- C1, C2, C3, C4, C5, C6, C7: footprint Capacitor_SMD:C_0805_2012Metric -> Capacitor_SMD:C_0603_1608Metric; moved to B.Cu
- D1, D10, D11, D12, D13, D14, D15, D16, D17, D18, D19, D2, D20, D21, D22, D23, D24, D25, D28, D29, D3, D30, D31, D32, D33, D34, D35, D36, D37, D38, D39, D4, D40, D41, D42, D43, D44, D5, D6, D7, D8, D9, F1, MX1, MX10, MX11, MX12, MX13, MX14, MX15, MX16, MX17, MX18, MX19, MX2, MX20, MX21, MX22, MX23, MX24, MX25, MX28, MX29, MX3, MX30, MX31, MX32, MX33, MX34, MX35, MX36, MX37, MX38, MX39, MX4, MX40, MX41, MX42, MX43, MX44, MX5, MX6, MX7, MX8, MX9, SW1, U1, USB1, Y1: moved to B.Cu
- R1, R2, R3, R4, R5, R6: footprint Resistor_SMD:R_0805_2012Metric -> Resistor_SMD:R_0603_1608Metric; moved to B.Cu
- moved MX44 215.5 mm to (40.9, 118.3), turned to 170 degrees
- moved MX33 215.5 mm to (256.4, 118.4), turned to 190 degrees
- moved D44 214.3 mm to (41.5, 110.4), turned to 170 degrees
- moved D33 211.2 mm to (254.3, 110.7), turned to 190 degrees
- moved MX32 208.9 mm to (44.2, 99.6), turned to 170 degrees
- moved MX21 208.9 mm to (253.1, 99.6), turned to 190 degrees
- moved D32 207.7 mm to (44.8, 91.6), turned to 170 degrees
- moved D21 205.3 mm to (251.4, 91.9), turned to 190 degrees
- moved MX20 202.3 mm to (47.5, 80.8), turned to 170 degrees
- moved MX11 202.3 mm to (249.8, 80.8), turned to 190 degrees
- moved D20 201.1 mm to (48.1, 72.9), turned to 170 degrees
- moved D11 198.0 mm to (247.7, 73.2), turned to 190 degrees
- moved MX10 195.7 mm to (50.8, 62.0), turned to 170 degrees
- moved MX1 195.7 mm to (246.5, 62.1), turned to 190 degrees
- moved D10 194.5 mm to (51.4, 54.1), turned to 170 degrees
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Connections:
- MX1 pad 1: Col0 -> Col11
- MX10 pad 1: Col11 -> Col0
- MX11 pad 1: Col0 -> Col11
- MX12 pad 1: Col1 -> Col10
- MX13 pad 1: Col2 -> Col9
- MX14 pad 1: Col3 -> Col8
- MX15 pad 1: Col4 -> Col7
- MX16 pad 1: Col7 -> Col4
- MX17 pad 1: Col8 -> Col3
- MX18 pad 1: Col9 -> Col2
- MX19 pad 1: Col10 -> Col1
- MX2 pad 1: Col1 -> Col10
- MX20 pad 1: Col11 -> Col0
- MX21 pad 1: Col0 -> Col11
- MX22 pad 1: Col1 -> Col10
- MX23 pad 1: Col2 -> Col9
- MX24 pad 1: Col3 -> Col8
- MX25 pad 1: Col4 -> Col7
- MX28 pad 1: Col7 -> Col4
- MX29 pad 1: Col8 -> Col3
- MX3 pad 1: Col2 -> Col9
- MX30 pad 1: Col9 -> Col2
- MX31 pad 1: Col10 -> Col1
- MX32 pad 1: Col11 -> Col0
- MX33 pad 1: Col0 -> Col11
- MX34 pad 1: Col1 -> Col10
- MX35 pad 1: Col2 -> Col9
- MX36 pad 1: Col3 -> Col8
- MX37 pad 1: Col4 -> Col7
- MX38 pad 1: Col5 -> Col6
- MX39 pad 1: Col6 -> Col5
- MX4 pad 1: Col3 -> Col8
- MX40 pad 1: Col7 -> Col4
- MX41 pad 1: Col8 -> Col3
- MX42 pad 1: Col9 -> Col2
- MX43 pad 1: Col10 -> Col1
- MX44 pad 1: Col11 -> Col0
- MX5 pad 1: Col4 -> Col7
- MX6 pad 1: Col7 -> Col4
- MX7 pad 1: Col8 -> Col3
- MX8 pad 1: Col9 -> Col2
- MX9 pad 1: Col10 -> Col1
- U1 pad 10: Col2 -> Net-(U1-Pad10)
- U1 pad 11: Col3 -> Net-(U1-Pad11)
- U1 pad 12: Col4 -> Net-(U1-Pad12)
- U1 pad 18: Net-(U1-Pad18) -> Col7
- U1 pad 19: Net-(U1-Pad19) -> Col8
- U1 pad 20: Net-(U1-Pad20) -> Col9
- U1 pad 21: Net-(U1-Pad21) -> Col10
- U1 pad 22: Col5 -> Col11
- U1 pad 25: Net-(U1-Pad25) -> Col6
- U1 pad 26: Net-(U1-Pad26) -> Col5
- U1 pad 36: Col6 -> Col0
- U1 pad 37: Col7 -> Col1
- U1 pad 38: Col8 -> Col2
- U1 pad 39: Col9 -> Col3
- U1 pad 40: Col10 -> Col4
- U1 pad 41: Col11 -> Net-(U1-Pad41)
- U1 pad 8: Col0 -> Net-(U1-Pad8)
- U1 pad 9: Col1 -> Net-(U1-Pad9)
Routing:
- net Row2: track 397.2 -> 321.2 mm
- net Row1: track 400.1 -> 359.0 mm
- net Row0: track 398.8 -> 360.7 mm
- net Row3: track 418.3 -> 389.1 mm
- net Col0: track 184.6 -> 167.7 mm
- net Col1: track 162.6 -> 147.3 mm
- net Net-(R1-Pad2): track 34.3 -> 19.9 mm
- net VCC: track 30.7 -> 16.6 mm
- net Col4: track 97.8 -> 83.9 mm
- net +5V: track 61.0 -> 74.8 mm
- net Col2: track 140.0 -> 126.8 mm
- net Col3: track 117.8 -> 105.3 mm
- net Net-(C3-Pad1): track 5.86 -> 12.4 mm
- net Col6: track 27.8 -> 32.0 mm
- net GND: track 127.7 -> 123.7 mm, vias 0 -> 2
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- removed copper zone on F.Cu, net (none)
- removed copper zone on F.Cu, net GND

Commit message: Complete reroute
Parts:
- MX1, MX10, MX11, MX12, MX13, MX14, MX15, MX16, MX17, MX18, MX19, MX2, MX20, MX21, MX22, MX23, MX24, MX25, MX28, MX29, MX3, MX30, MX31, MX32, MX33, MX34, MX35, MX36, MX37, MX38, MX39, MX4, MX40, MX41, MX42, MX43, MX44, MX5, MX6, MX7, MX8, MX9: moved to F.Cu
- moved MX33 224.7 mm to (31.9, 125.7), turned to 350 degrees
- moved D33 220.3 mm to (34.0, 118.0), turned to 350 degrees
- moved MX21 218.0 mm to (35.2, 106.9), turned to 350 degrees
- moved D21 214.5 mm to (37.0, 99.2), turned to 350 degrees
- moved MX11 211.4 mm to (38.5, 88.1), turned to 350 degrees
- moved D11 207.1 mm to (40.7, 80.5), turned to 350 degrees
- moved MX44 206.6 mm to (247.4, 125.6), turned to 10 degrees
- moved D44 205.4 mm to (246.8, 117.7), turned to 10 degrees
- moved MX1 204.8 mm to (41.8, 69.4), turned to 350 degrees
- moved D1 200.5 mm to (44.0, 61.7), turned to 350 degrees
- moved MX32 200.0 mm to (244.1, 106.9), turned to 10 degrees
- moved D32 198.8 mm to (243.5, 98.9), turned to 10 degrees
- moved MX20 193.4 mm to (240.8, 88.1), turned to 10 degrees
- moved D20 192.2 mm to (240.2, 80.2), turned to 10 degrees
- moved MX10 186.8 mm to (237.5, 69.3), turned to 10 degrees
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Connections:
- MX1 pad 1: Col11 -> Col0
- MX10 pad 1: Col0 -> Col11
- MX11 pad 1: Col11 -> Col0
- MX12 pad 1: Col10 -> Col1
- MX13 pad 1: Col9 -> Col2
- MX14 pad 1: Col8 -> Col3
- MX15 pad 1: Col7 -> Col4
- MX16 pad 1: Col4 -> Col7
- MX17 pad 1: Col3 -> Col8
- MX18 pad 1: Col2 -> Col9
- MX19 pad 1: Col1 -> Col10
- MX2 pad 1: Col10 -> Col1
- MX20 pad 1: Col0 -> Col11
- MX21 pad 1: Col11 -> Col0
- MX22 pad 1: Col10 -> Col1
- MX23 pad 1: Col9 -> Col2
- MX24 pad 1: Col8 -> Col3
- MX25 pad 1: Col7 -> Col4
- MX28 pad 1: Col4 -> Col7
- MX29 pad 1: Col3 -> Col8
- MX3 pad 1: Col9 -> Col2
- MX30 pad 1: Col2 -> Col9
- MX31 pad 1: Col1 -> Col10
- MX32 pad 1: Col0 -> Col11
- MX33 pad 1: Col11 -> Col0
- MX34 pad 1: Col10 -> Col1
- MX35 pad 1: Col9 -> Col2
- MX36 pad 1: Col8 -> Col3
- MX37 pad 1: Col7 -> Col4
- MX38 pad 1: Col6 -> Col5
- MX39 pad 1: Col5 -> Col6
- MX4 pad 1: Col8 -> Col3
- MX40 pad 1: Col4 -> Col7
- MX41 pad 1: Col3 -> Col8
- MX42 pad 1: Col2 -> Col9
- MX43 pad 1: Col1 -> Col10
- MX44 pad 1: Col0 -> Col11
- MX5 pad 1: Col7 -> Col4
- MX6 pad 1: Col4 -> Col7
- MX7 pad 1: Col3 -> Col8
- MX8 pad 1: Col2 -> Col9
- MX9 pad 1: Col1 -> Col10
Routing:
- net Row2: track 321.2 -> 274.4 mm
- net Row1: track 359.0 -> 380.3 mm
- net Row0: track 360.7 -> 379.9 mm
- net Col2: track 126.8 -> 140.2 mm, vias 1 -> 0
- net Col4: track 83.9 -> 97.4 mm, vias 1 -> 0
- net Col3: track 105.3 -> 118.0 mm, vias 1 -> 0
- net Col0: track 167.7 -> 178.1 mm, vias 1 -> 0
- net Col1: track 147.3 -> 156.4 mm, vias 1 -> 0
- net Col5: track 29.3 -> 37.7 mm
- net Col11: track 177.6 -> 170.8 mm, vias 1 -> 0
- net Col6: track 32.0 -> 26.2 mm
- net GND: track 123.7 -> 129.2 mm
- net Col10: track 153.8 -> 148.5 mm, vias 1 -> 0
- net Row3: track 389.1 -> 386.7 mm
- net +5V: track 74.8 -> 72.6 mm, vias 4 -> 5
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- added copper zone on B.Cu, net (none)
- added copper zone on B.Cu, net GND
- added copper zone on F.Cu, net GND
Other:
- outline, holes or cut-outs redrawn

Commit message: Small Updates
- Decoupled USB Shield from GND
- Cap to GND as a LPF for the RST button
- Copper layer cleanup
- Rounded PCB corners
Parts:
- added C8: 100nF, Capacitor_SMD:C_0603_1608Metric, B.Cu at (146.8, 83.2)
- added C9: 100nF, Capacitor_SMD:C_0603_1608Metric, B.Cu at (148.5, 95.4)
- added R7: 1M, Resistor_SMD:R_0603_1608Metric, B.Cu at (144.8, 83.2)
Connections:
- USB1 pad 13: GND -> Net-(C8-Pad2)
Routing:
- net GND: track 129.2 -> 193.9 mm, vias 2 -> 13
- net Net-(C8-Pad2): track 0.00 -> 7.60 mm
- net Net-(C9-Pad1): track 19.8 -> 21.7 mm
- removed copper zone on B.Cu, net (none)
Other:
- board size 240.3 x 101.9 mm -> 238.8 x 97.8 mm
