File: Marv-Atreus.kicad_pcb (KiCad board)
At the start: 2 copper layers, 238.8 x 97.8 mm, 105 parts, among them SW1 SW_Push, U1 ATmega32U4-AU, Y1 16MHz

Commit message: Even more Updates
- switched from Crystal to resonator
- added ESD protection ic
- Cleaned up silkscreen
Parts:
- removed C1, C2: 22pF, Capacitor_SMD:C_0603_1608Metric
- added U2: USBLC6-2SC6, Package_TO_SOT_SMD:SOT-23-6, B.Cu at (139.7, 83.6)
- D1, D10, D11, D12, D13, D14, D15, D16, D17, D18, D19, D2, D20, D21, D22, D23, D24, D25, D28, D29, D3, D30, D31, D32, D33, D34, D35, D36, D37, D38, D39, D4, D40, D41, D42, D43, D44, D5, D6, D7, D8, D9: footprint Diode_SMD:D_SOD-123 -> random-keyboard-parts:D_SOD-123_NoReference
- Y1: value 16MHz -> Resonator_Small; footprint Crystal:Crystal_SMD_3225-4Pin_3.2x2.5mm -> Crystal:Resonator_SMD_muRata_CSTxExxV-3Pin_3.0x1.1mm
- moved R5 5.21 mm to (140.7, 88.0)
- moved R4 5.18 mm to (138.8, 88.0)
- moved SW1 2.29 mm to (144.7, 89.9), turned to 90 degrees
- moved Y1 2.15 mm to (149.8, 106.0)
- moved C7 2.11 mm to (140.9, 97.7)
- moved C4 1.92 mm to (133.3, 100.0)
- moved C6 1.92 mm to (133.3, 112.9)
- moved C3 1.92 mm to (146.2, 99.9)
- moved C5 1.92 mm to (146.1, 112.8)
- moved C9 1.92 mm to (148.8, 97.4)
- moved R1 1.92 mm to (147.5, 98.6)
- moved R6 1.92 mm to (132.0, 114.1)
- moved U1 1.92 mm to (139.7, 106.4)
- moved F1 0.07 mm to (134.3, 84.0)
Connections:
- net Net-(U1-Pad41) renamed LedSig
- R4 pad 2: D+ -> Net-(R4-Pad2)
- R5 pad 2: D- -> Net-(R5-Pad2)
- U1 pad 3: Net-(R5-Pad1) -> Net-(R4-Pad1)
- U1 pad 4: Net-(R4-Pad1) -> Net-(R5-Pad1)
Routing:
- net GND: track 193.9 -> 98.5 mm, vias 13 -> 12
- net Net-(C9-Pad1): track 21.7 -> 13.3 mm
- net Net-(U1-Pad16): track 10.8 -> 4.76 mm
- net VCC: track 17.8 -> 22.6 mm, vias 0 -> 2
- net Net-(R4-Pad1): track 16.5 -> 12.5 mm
- net Net-(U1-Pad17): track 8.33 -> 4.74 mm
- net Net-(R4-Pad2): track 0.00 -> 2.48 mm
- net Net-(R5-Pad2): track 0.00 -> 2.46 mm
- net Col5: track 37.7 -> 35.7 mm
- net Col6: track 26.2 -> 24.4 mm
- net +5V: track 72.6 -> 74.2 mm
- net Net-(R5-Pad1): track 15.6 -> 14.0 mm
- net Col8: track 110.1 -> 108.7 mm
- net Col11: track 170.8 -> 169.8 mm
- net Col9: track 132.0 -> 131.1 mm
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
Commit message: Added ISP Connector
Parts:
- added J1: Conn_02x03_Odd_Even, Connector_PinHeader_2.54mm:PinHeader_2x03_P2.54mm_Vertical, B.Cu at (154.3, 106.5)
Connections:
- net Net-(C9-Pad1) renamed RST
- U1 pad 10: Net-(U1-Pad10) -> MOSI
- U1 pad 11: Net-(U1-Pad11) -> MISO
- U1 pad 9: Net-(U1-Pad9) -> SCK
Routing:
- net SCK: track 0.00 -> 35.2 mm, vias 0 -> 1
- net MOSI: track 0.00 -> 22.5 mm, vias 0 -> 1
- net MISO: track 0.00 -> 22.2 mm, vias 0 -> 1
- net +5V: track 74.2 -> 84.5 mm
- net RST: track 13.3 -> 23.3 mm, vias 0 -> 1

Commit message: Updates
- Added TVS diode to vbus
- Reinforced power lines
- More cleanup
Parts:
- added D26: TVS 5V, Diode_SMD:D_SMB, B.Cu at (130.6, 85.4)
Connections:
- U2 pad 5: VCC -> Net-(U2-Pad5)
Routing:
- net VCC: track 22.6 -> 16.1 mm, vias 2 -> 0
- net GND: track 98.5 -> 92.8 mm, vias 12 -> 14
- net Row1: track 380.9 -> 383.0 mm
- net Net-(R4-Pad1): track 12.5 -> 13.7 mm
- net Net-(R5-Pad1): track 14.0 -> 13.0 mm

Commit message: Layout Updates
Parts:
- moved D26 9.61 mm to (135.1, 93.9)
Routing:
- net VCC: track 16.1 -> 24.4 mm
- net +5V: track 84.5 -> 87.4 mm
Changed lines of the file:
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@@
     (thickness 1.6)
     (drawings 203)
-    (tracks 911)
+    (tracks 915)
     (zones 0)
     (modules 106)
@@
   )
   (module Diode_SMD:D_SMB (layer B.Cu)
-    (at 130.633 85.412 270)
+    (at 135.078 93.93 270)
     (descr "Diode SMB (DO-214AA)")
     (tags "Diode SMB (DO-214AA)")
@@
   (segment (start 133.824 111.125897) (end 133.831096 111.132993) (width 0.25) (layer F.Cu) (net 3))
   (segment (start 133.824 101.271) (end 133.824 111.125897) (width 0.6) (layer F.Cu) (net 3))
-  (segment (start 136.602 96.652124) (end 133.824 99.430124) (width 0.6) (layer B.Cu) (net 3))
-  (segment (start 134.316 85.666) (end 134.189 85.793) (width 0.6) (layer B.Cu) (net 3))
-  (segment (start 134.316 85.412) (end 134.316 85.666) (width 0.6) (layer B.Cu) (net 3))
-  (segment (start 134.189 85.793) (end 134.189 85.91) (width 0.6) (layer B.Cu) (net 3))
-  (segment (start 134.189 85.91) (end 136.602 88.323) (width 0.6) (layer B.Cu) (net 3))
-  (segment (start 136.602 88.323) (end 136.602 96.652124) (width 0.6) (layer B.Cu) (net 3))
   (segment (start 135.586 102.303) (end 141.493884 102.303) (width 0.6) (layer F.Cu) (net 3))
   (segment (start 143.267116 104.076232) (end 143.968 104.076232) (width 0.6) (layer F.Cu) (net 3))
@@
   (segment (start 133.808 111.109897) (end 133.831096 111.132993) (width 0.4) (layer B.Cu) (net 3))
   (segment (start 133.808 110.583925) (end 133.808 111.109897) (width 0.4) (layer B.Cu) (net 3))
+  (segment (start 134.316 85.666) (end 134.189 85.793) (width 0.6) (layer B.Cu) (net 3))
+  (segment (start 134.189 85.91) (end 138.126 89.847) (width 0.6) (layer B.Cu) (net 3))
+  (segment (start 138.126 97.985) (end 136.680876 99.430124) (width 0.6) (layer B.Cu) (net 3))
+  (segment (start 134.316 85.412) (end 134.316 85.666) (width 0.6) (layer B.Cu) (net 3))
+  (segment (start 136.680876 99.430124) (end 133.824 99.430124) (width 0.6) (layer B.Cu) (net 3))
+  (segment (start 138.126 89.847) (end 138.126 97.985) (width 0.6) (layer B.Cu) (net 3))
+  (segment (start 134.189 85.793) (end 134.189 85.91) (width 0.6) (layer B.Cu) (net 3))
   (segment (start 45.594915 64.420346) (end 45.193498 64.821763) (width 0.25) (layer B.Cu) (net 4))
   (segment (start 45.594915 61.990941) (end 45.594915 64.420346) (width 0.25) (layer B.Cu) (net 4))
@@
   (segment (start 142.102503 77.958503) (end 142.102503 78.853648) (width 0.25) (layer B.Cu) (net 50))
   (segment (start 137.202503 78.093646) (end 137.942512 77.353637) (width 0.25) (layer B.Cu) (net 50))
-  (segment (start 131.283 82.612) (end 130.633 83.262) (width 0.25) (layer B.Cu) (net 50))
-  (segment (start 134.316 82.612) (end 131.283 82.612) (width 0.7) (layer B.Cu) (net 50))
+  (segment (start 132.538 90.64) (end 133.678 91.78) (width 0.7) (layer B.Cu) (net 50))
+  (segment (start 132.538 83.515) (end 132.538 90.64) (width 0.7) (layer B.Cu) (net 50))
+  (segment (start 134.316 82.612) (end 133.441 82.612) (width 0.7) (layer B.Cu) (net 50))
+  (segment (start 133.678 91.78) (end 135.078 91.78) (width 0.7) (layer B.Cu) (net 50))
+  (segment (start 133.441 82.612) (end 132.538 83.515) (width 0.7) (layer B.Cu) (net 50))
   (segment (start 38.498903 81.673138) (end 35.190897 84.981144) (width 0.25) (layer F.Cu) (net 51))
   (segment (start 38.498903 66.220509) (end 38.498903 81.673138) (width 0.25) (layer F.Cu) (net 51))

Commit message: v0.1
Hopefully its a working pcb :baby_chick:
Routing:
- net Col3: track 117.3 -> 116.3 mm
- net Row2: track 275.4 -> 276.0 mm
- net Col1: track 155.8 -> 155.2 mm
- net Col2: track 139.5 -> 139.0 mm
- net GND: vias 14 -> 15
